File: pcb/logic.brd (EAGLE design)
At the start: 44.5 x 57.1 mm, 36 parts, among them SW1 FSM4JSMA, U1 LD1117, U2 MIC29302AWD

Commit message: Fixed resistor values
Parts:
- R1: value 150 -> 383
- R2: value 562 -> 100
Other:
- board text added: "Teensy 3.1"
- board text removed: "Teensy 3.0"
Changed lines of the file:
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@@
 <text x="2.54" y="9.2075" size="1.778" layer="21" align="center-left">+</text>
 <text x="11.1125" y="9.2075" size="1.778" layer="21" align="center-left">-</text>
-<text x="34.29" y="19.05" size="1.778" layer="21" rot="R90" align="center">Teensy 3.0</text>
+<text x="34.29" y="19.05" size="1.778" layer="21" rot="R90" align="center">Teensy 3.1</text>
 <text x="33.02" y="40.9575" size="1.27" layer="21" rot="R90">nRF24L01+</text>
 <text x="15.875" y="54.61" size="0.8128" layer="21" align="center">GND</text>
@@
 </element>
 <element name="JP1" library="SparkFun-Connectors" package="SCREWTERMINAL-5MM-2" value="M025MM" x="5.08" y="3.81" smashed="yes"/>
-<element name="R1" library="SparkFun-Passives" package="0603-RES" value="150" x="13.97" y="27.305" rot="R180"/>
-<element name="R2" library="SparkFun-Passives" package="0603-RES" value="562" x="15.24" y="24.765" rot="R180"/>
+<element name="R1" library="SparkFun-Passives" package="0603-RES" value="383" x="13.97" y="27.305" rot="R180"/>
+<element name="R2" library="SparkFun-Passives" package="0603-RES" value="100" x="15.24" y="24.765" rot="R180"/>
 <element name="C5" library="SparkFun-Passives" package="CPOL-RADIAL-10UF-25V" value="22uF" x="15.5575" y="20.32" smashed="yes" rot="R270">
 <attribute name="NAME" x="17.7165" y="17.7165" size="0.8128" layer="25" ratio="10"/>

Commit message: Updated resistor values
Parts:
- R3: value 132 -> 150
- R5, R6, R7, R8: value 681 -> 332
- R9: value 681 -> 200
Changed lines of the file:
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@@
 <attribute name="PROD_ID" value="TRANS-08345" x="13.97" y="44.1325" size="1.778" layer="27" rot="R90" display="off"/>
 </element>
-<element name="R3" library="SparkFun-Passives" package="0603-RES" value="132" x="18.415" y="41.5925" rot="R180"/>
+<element name="R3" library="SparkFun-Passives" package="0603-RES" value="150" x="18.415" y="41.5925" rot="R180"/>
 <element name="R4" library="SparkFun-Passives" package="0603-RES" value="100K" x="16.51" y="44.1325" rot="R270"/>
 <element name="STANDOFF2" library="SparkFun-Electromechanical" package="STAND-OFF" value="STAND-OFF" x="19.05" y="3.81"/>
@@
 <element name="LED4" library="SparkFun-LED" package="LED-0603" value="" x="20.32" y="20.32" rot="R90"/>
 <element name="LED5" library="SparkFun-LED" package="LED-0603" value="" x="14.605" y="6.0325" rot="R180"/>
-<element name="R5" library="SparkFun-Passives" package="0603-RES" value="681" x="30.48" y="17.78" rot="R180"/>
-<element name="R6" library="SparkFun-Passives" package="0603-RES" value="681" x="30.48" y="15.24" rot="R180"/>
-<element name="R7" library="SparkFun-Passives" package="0603-RES" value="681" x="30.48" y="12.7" rot="R180"/>
-<element name="R8" library="SparkFun-Passives" package="0603-RES" value="681" x="30.48" y="10.16" rot="R180"/>
-<element name="R9" library="SparkFun-Passives" package="0603-RES" value="681" x="14.605" y="2.54" rot="R90"/>
+<element name="R5" library="SparkFun-Passives" package="0603-RES" value="332" x="30.48" y="17.78" rot="R180"/>
+<element name="R6" library="SparkFun-Passives" package="0603-RES" value="332" x="30.48" y="15.24" rot="R180"/>
+<element name="R7" library="SparkFun-Passives" package="0603-RES" value="332" x="30.48" y="12.7" rot="R180"/>
+<element name="R8" library="SparkFun-Passives" package="0603-RES" value="332" x="30.48" y="10.16" rot="R180"/>
+<element name="R9" library="SparkFun-Passives" package="0603-RES" value="200" x="14.605" y="2.54" rot="R90"/>
 </elements>
 <signals>
